File: Electronics/GhostS-PCB/GhostS-PCB.kicad_pcb (KiCad board)
At the start: 2 copper layers, 289 x 103 mm, 404 parts, among them IC1 IP5306_4.35V, IC2 DW01, J1 Conn_01x06_Female, J2 Conn_01x08_Female, J3 USB_C_Receptacle_USB2.0, J4 Cell+, J5 Cell-, K1 KEYSW, K10 KEYSW, K11 KEYSW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

Commit message: .
Other:
- net class Default removed
- net class Power removed
